Commit message: Load diff controller correctly and fix imu name

File: wheeled_biped_description/models/model.gazebo.xacro (robot description, xacro)
@@ -7,6 +7,6 @@
   </gazebo>
   <gazebo reference="imu_link">
-    <sensor name='imu_gnss' type='imu'>
-      <topic>/imu</topic>
+    <sensor name='imu_head' type='imu'>
+      <topic>/imu/head</topic>
       <update_rate>200</update_rate>
       <always_on>true</always_on>

File: wheeled_biped_description/models/model.urdf.xacro (robot description, xacro)
@@ -4,8 +4,8 @@
   <xacro:property name="head_mass" value="0.250" />
   <xacro:property name="head_height" value="0.05" />
-  <xacro:property name="head_size" value="0.100" />
+  <xacro:property name="head_size" value="0.100" /> <!-- WARNING: Also edit controllers.yaml wheel_separation -->
   <xacro:property name="joint_mass" value="0.100" />
   <xacro:property name="knee_height" value="0.150" /> <!-- From this is the thigh length -->
-  <xacro:property name="wheel_radius" value="0.025" />
+  <xacro:property name="wheel_radius" value="0.025" /> <!-- WARNING: Also edit controllers.yaml wheel_radius -->
   <xacro:property name="wheel_length" value="0.025" />
   <xacro:property name="wheel_mass" value="0.100" />
