Commit message: Add knee controllers and update screenshot

File: wheeled_biped_description/models/model.urdf.xacro (robot description, xacro)
@@ -93,5 +93,6 @@
     <axis xyz="0 0 1"/>
     <dynamics damping="0.5"/>
-    <limit lower="0" upper="${pi}" effort="30" velocity="${pi}"/>
+    <!-- Negative is forwards, because of the right hand rule on the joint -->
+    <limit lower="${-(pi/2 + pi/4)}" upper="0" effort="100" velocity="1.0"/>
   </joint>
   <link name="lower_left_leg_link">
@@ -164,5 +165,6 @@
     <axis xyz="0 0 1"/>
     <dynamics damping="0.5"/>
-    <limit lower="0" upper="${pi}" effort="30" velocity="${pi}"/>
+    <!-- Negative is forwards, because of the right hand rule on the joint -->
+    <limit lower="${-(pi/2 + pi/4)}" upper="0" effort="100" velocity="1.0"/>
   </joint>
   <link name="lower_right_leg_link">

File: wheeled_biped_description/models/ros2_control.xacro (robot description, xacro)
@@ -14,4 +14,22 @@
       </xacro:unless>
     </hardware>
+    <joint name="lower_left_leg_joint">
+      <command_interface name="position">
+        <!-- Negative is forwards, because of the right hand rule on the joint -->
+        <param name="min">${-(pi/2 + pi/4)}</param>
+        <!-- 0 means the leg is extended -->
+        <param name="max">0</param>
+      </command_interface>
+      <state_interface name="position"/>
+    </joint>
+    <joint name="lower_right_leg_joint">
+      <command_interface name="position">
+        <!-- Negative is forwards, because of the right hand rule on the joint -->
+        <param name="min">${-(pi/2 + pi/4)}</param>
+        <!-- 0 means the leg is extended -->
+        <param name="max">0</param>
+      </command_interface>
+      <state_interface name="position"/>
+    </joint>
     <joint name="left_wheel_joint">
       <command_interface name="velocity"/>

Commit message: Add controllers for the hips

File: wheeled_biped_description/models/model.urdf.xacro (robot description, xacro)
@@ -69,5 +69,5 @@
     <axis xyz="0 0 1"/>
     <dynamics damping="0.5"/>
-    <limit lower="0" upper="${pi/2}" effort="30" velocity="${pi}"/>
+    <limit lower="${-pi/2}" upper="${pi/2}" effort="100" velocity="1.0"/>
   </joint>
   <link name="upper_left_leg_link">
@@ -135,5 +135,5 @@
     </xacro:inertial_cylinder>
   </link>
-    <joint name="upper_right_leg_joint" type="revolute">
+  <joint name="upper_right_leg_joint" type="revolute">
     <parent link="head_link"/>
     <child link="upper_right_leg_link"/>
@@ -141,5 +141,5 @@
     <axis xyz="0 0 1"/>
     <dynamics damping="0.5"/>
-    <limit lower="0" upper="${pi/2}" effort="30" velocity="${pi}"/>
+    <limit lower="${-pi/2}" upper="${pi/2}" effort="100" velocity="1.0"/>
   </joint>
   <link name="upper_right_leg_link">

File: wheeled_biped_description/models/ros2_control.xacro (robot description, xacro)
@@ -14,4 +14,22 @@
       </xacro:unless>
     </hardware>
+    <!-- Hips -->
+    <joint name="upper_left_leg_joint">
+      <command_interface name="position">
+        <!-- Negative is forwards, because of the right hand rule on the joint -->
+        <param name="min">${-(pi/2)}</param>
+        <param name="max">${pi/2}</param>
+      </command_interface>
+      <state_interface name="position"/>
+    </joint>
+    <joint name="upper_right_leg_joint">
+      <command_interface name="position">
+        <!-- Negative is forwards, because of the right hand rule on the joint -->
+        <param name="min">${-(pi/2)}</param>
+        <param name="max">${pi/2}</param>
+      </command_interface>
+      <state_interface name="position"/>
+    </joint>
+    <!-- Knees -->
     <joint name="lower_left_leg_joint">
       <command_interface name="position">
@@ -32,4 +50,5 @@
       <state_interface name="position"/>
     </joint>
+    <!-- Wheels -->
     <joint name="left_wheel_joint">
       <command_interface name="velocity"/>
